File: IO4-SignalDriver-Small.brd (EAGLE design)
At the start: 50 x 43.6 mm, 17 parts, among them IC1 74HS139A

Commit message: added values for connectors
Parts:
- CON4, CON5: value (none) -> 3.5mm
- HEAD1: value Head 1 -> 2mm
- HEAD2: value Head 2 -> 2mm
- IO4: value (none) -> RJ12/6
Changed lines of the file:
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@@
 <attribute name="NAME" x="18.653" y="34.0995" size="0.4064" layer="25"/>
 </element>
-<element name="IO4" library="SPCoast" package="RJ25-INVERTED" value="" x="44.815" y="21.59" smashed="yes" rot="R90">
+<element name="IO4" library="SPCoast" package="RJ25-INVERTED" value="RJ12/6" x="44.815" y="21.59" smashed="yes" rot="R90">
 <attribute name="NAME" x="38.211" y="19.05" size="1.778" layer="25" rot="R90"/>
 <attribute name="VALUE" x="34.655" y="16.637" size="1.778" layer="27" rot="R90"/>
 </element>
-<element name="CON4" library="SPCoast" package="SCREWTERMINAL-3.5MM-4" value="" x="3.54" y="18.415" rot="R270"/>
-<element name="CON5" library="SPCoast" package="SCREWTERMINAL-3.5MM-4" value="" x="3.54" y="35.941" rot="R270"/>
-<element name="HEAD1" library="SPCoast" package="4P-2.0" value="Head 1" x="9.89" y="29.845" smashed="yes" rot="R270">
+<element name="CON4" library="SPCoast" package="SCREWTERMINAL-3.5MM-4" value="3.5mm" x="3.54" y="18.415" rot="R270"/>
+<element name="CON5" library="SPCoast" package="SCREWTERMINAL-3.5MM-4" value="3.5mm" x="3.54" y="35.941" rot="R270"/>
+<element name="HEAD1" library="SPCoast" package="4P-2.0" value="2mm" x="9.89" y="29.845" smashed="yes" rot="R270">
 <attribute name="NAME" x="8.62" y="23.495" size="0.889" layer="25" font="vector" ratio="11"/>
 </element>
-<element name="HEAD2" library="SPCoast" package="4P-2.0" value="Head 2" x="9.89" y="13.97" smashed="yes" rot="R270">
+<element name="HEAD2" library="SPCoast" package="4P-2.0" value="2mm" x="9.89" y="13.97" smashed="yes" rot="R270">
 <attribute name="NAME" x="8.62" y="7.62" size="0.889" layer="25" font="vector" ratio="11"/>
 </element>

Commit message: normalized values
Parts:
- C1: device SPCoast:0805-CAP -> SPCoast:0603-CAP
- R10, R4, R6, R7, R8, R9: device SPCoast:0805-RES -> SPCoast:0603-RES
Changed lines of the file:
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@@
 <attribute name="NAME" x="32.369" y="13.589" size="1.27" layer="25" ratio="10" rot="R90"/>
 </element>
-<element name="C1" library="SPCoast" package="0805-CAP" value="0.1UF" x="23.225" y="21.336" smashed="yes" rot="R270">
+<element name="C1" library="SPCoast" package="0603-CAP" value="0.1UF" x="23.225" y="21.336" smashed="yes" rot="R270">
 <attribute name="NAME" x="22.717" y="23.241" size="0.8128" layer="25"/>
 <attribute name="VALUE" x="23.733" y="25.781" size="0.8128" layer="27"/>
 </element>
-<element name="R4" library="SPCoast" package="0805-RES" value="1k0" x="19.415" y="14.224" smashed="yes">
+<element name="R4" library="SPCoast" package="0603-RES" value="1k0" x="19.415" y="14.224" smashed="yes">
 <attribute name="NAME" x="18.653" y="15.0495" size="0.4064" layer="25"/>
 <attribute name="VALUE" x="24.495" y="30.734" size="0.8128" layer="27"/>
 </element>
-<element name="R6" library="SPCoast" package="0805-RES" value="2k2" x="19.415" y="10.414" smashed="yes">
+<element name="R6" library="SPCoast" package="0603-RES" value="2k2" x="19.415" y="10.414" smashed="yes">
 <attribute name="NAME" x="18.653" y="11.2395" size="0.4064" layer="25"/>
 <attribute name="VALUE" x="24.495" y="27.559" size="0.8128" layer="27"/>
 </element>
-<element name="R7" library="SPCoast" package="0805-RES" value="2k2" x="19.415" y="18.034" smashed="yes">
+<element name="R7" library="SPCoast" package="0603-RES" value="2k2" x="19.415" y="18.034" smashed="yes">
 <attribute name="NAME" x="18.653" y="18.8595" size="0.4064" layer="25"/>
 <attribute name="VALUE" x="24.495" y="34.544" size="0.8128" layer="27"/>
 </element>
-<element name="R8" library="SPCoast" package="0805-RES" value="1k0" x="19.415" y="30.099" smashed="yes">
+<element name="R8" library="SPCoast" package="0603-RES" value="1k0" x="19.415" y="30.099" smashed="yes">
 <attribute name="NAME" x="18.653" y="30.9245" size="0.4064" layer="25"/>
 </element>
-<element name="R9" library="SPCoast" package="0805-RES" value="2k2" x="19.415" y="26.924" smashed="yes">
+<element name="R9" library="SPCoast" package="0603-RES" value="2k2" x="19.415" y="26.924" smashed="yes">
 <attribute name="NAME" x="18.653" y="27.7495" size="0.4064" layer="25"/>
 </element>
-<element name="R10" library="SPCoast" package="0805-RES" value="2k2" x="19.415" y="33.274" smashed="yes">
+<element name="R10" library="SPCoast" package="0603-RES" value="2k2" x="19.415" y="33.274" smashed="yes">
 <attribute name="NAME" x="18.653" y="34.0995" size="0.4064" layer="25"/>
 </element>
@@
 <wire x1="26.273" y1="22.733" x2="25.003" y2="21.463" width="0.254" layer="1"/>
 <wire x1="25.003" y1="21.463" x2="25.003" y2="18.1356" width="0.254" layer="1"/>
-<wire x1="23.225" y1="20.436" x2="23.236" y2="20.447" width="0.254" layer="1"/>
+<wire x1="23.225" y1="20.486" x2="23.236" y2="20.447" width="0.254" layer="1"/>
 <via x="23.352" y="17.907" extent="1-16" drill="0.7"/>
 <wire x1="23.236" y1="20.447" x2="23.352" y2="20.331" width="0.4064" layer="1"/>
@@
 <contactref element="IC1" pad="16"/>
 <contactref element="C1" pad="1"/>
-<wire x1="23.225" y1="22.236" x2="24.379" y2="22.236" width="0.3048" layer="1"/>
+<wire x1="23.225" y1="22.186" x2="24.379" y2="22.236" width="0.3048" layer="1"/>
 <wire x1="24.379" y1="22.236" x2="25.003" y2="22.86" width="0.3048" layer="1"/>
 <wire x1="25.003" y1="22.86" x2="25.003" y2="24.2824" width="0.3048" layer="1"/>
-<wire x1="23.214" y1="22.225" x2="23.225" y2="22.236" width="0.3048" layer="1"/>
+<wire x1="23.214" y1="22.225" x2="23.225" y2="22.186" width="0.3048" layer="1"/>
 <polygon width="0.3048" layer="1" isolate="0.3048">
 <vertex x="0" y="0"/>
@@
 <contactref element="HEAD1" pad="2"/>
 <wire x1="9.636" y1="30.845" x2="10.382" y2="30.099" width="0.3048" layer="1"/>
-<wire x1="10.382" y1="30.099" x2="18.515" y2="30.099" width="0.3048" layer="1"/>
+<wire x1="10.382" y1="30.099" x2="18.565" y2="30.099" width="0.3048" layer="1"/>
 <wire x1="3.54" y1="32.441" x2="8.04" y2="32.441" width="0.4064" layer="16"/>
 <wire x1="8.04" y1="32.441" x2="9.636" y2="30.845" width="0.4064" layer="16"/>
@@
 <contactref element="HEAD2" pad="1"/>
 <wire x1="10.144" y1="16.97" x2="11.208" y2="18.034" width="0.3048" layer="1"/>
-<wire x1="11.208" y1="18.034" x2="18.515" y2="18.034" width="0.3048" layer="1"/>
+<wire x1="11.208" y1="18.034" x2="18.565" y2="18.034" width="0.3048" layer="1"/>
 <wire x1="3.54" y1="18.415" x2="8.699" y2="18.415" width="0.4064" layer="16"/>
 <wire x1="8.699" y1="18.415" x2="10.144" y2="16.97" width="0.4064" layer="16"/>
@@
 <contactref element="HEAD2" pad="3"/>
 <wire x1="10.144" y1="12.97" x2="12.7" y2="10.414" width="0.3048" layer="1"/>
-<wire x1="12.7" y1="10.414" x2="18.515" y2="10.414" width="0.3048" layer="1"/>
+<wire x1="12.7" y1="10.414" x2="18.565" y2="10.414" width="0.3048" layer="1"/>
 <wire x1="10.144" y1="12.97" x2="5.095" y2="12.97" width="0.4064" layer="16"/>
 <wire x1="5.095" y1="12.97" x2="3.54" y2="11.415" width="0.4064" layer="16"/>
@@
 <contactref element="HEAD2" pad="2"/>
 <wire x1="9.636" y1="14.97" x2="10.382" y2="14.224" width="0.3048" layer="1"/>
-<wire x1="10.382" y1="14.224" x2="18.515" y2="14.224" width="0.3048" layer="1"/>
+<wire x1="10.382" y1="14.224" x2="18.565" y2="14.224" width="0.3048" layer="1"/>
 <wire x1="9.636" y1="14.97" x2="3.595" y2="14.97" width="0.4064" layer="16"/>
 <wire x1="3.595" y1="14.97" x2="3.54" y2="14.915" width="0.4064" layer="16"/>
@@
 <contactref element="HEAD1" pad="1"/>
 <wire x1="10.144" y1="32.845" x2="10.573" y2="33.274" width="0.3048" layer="1"/>
-<wire x1="10.573" y1="33.274" x2="18.515" y2="33.274" width="0.3048" layer="1"/>
+<wire x1="10.573" y1="33.274" x2="18.565" y2="33.274" width="0.3048" layer="1"/>
 <wire x1="3.54" y1="35.941" x2="7.048" y2="35.941" width="0.4064" layer="16"/>
 <wire x1="7.048" y1="35.941" x2="10.144" y2="32.845" width="0.4064" layer="16"/>
@@
 <contactref element="HEAD1" pad="3"/>
 <wire x1="10.144" y1="28.845" x2="12.065" y2="26.924" width="0.3048" layer="1"/>
-<wire x1="12.065" y1="26.924" x2="18.515" y2="26.924" width="0.3048" layer="1"/>
+<wire x1="12.065" y1="26.924" x2="18.565" y2="26.924" width="0.3048" layer="1"/>
 <wire x1="3.54" y1="28.941" x2="10.048" y2="28.941" width="0.4064" layer="16"/>
 <wire x1="10.048" y1="28.941" x2="10.144" y2="28.845" width="0.4064" layer="16"/>
@@
 <wire x1="33.258" y1="22.86" x2="33.258" y2="26.924" width="0.2032" layer="1"/>
 <wire x1="33.258" y1="26.924" x2="26.908" y2="33.274" width="0.3048" layer="1"/>
-<wire x1="26.908" y1="33.274" x2="20.315" y2="33.274" width="0.3048" layer="1"/>
+<wire x1="26.908" y1="33.274" x2="20.265" y2="33.274" width="0.3048" layer="1"/>
 </signal>
 <signal name="R1">
@@
 <wire x1="29.448" y1="22.86" x2="29.448" y2="25.908" width="0.2032" layer="1"/>
 <wire x1="29.448" y1="25.908" x2="28.432" y2="26.924" width="0.3048" layer="1"/>
-<wire x1="28.432" y1="26.924" x2="20.315" y2="26.924" width="0.3048" layer="1"/>
+<wire x1="28.432" y1="26.924" x2="20.265" y2="26.924" width="0.3048" layer="1"/>
 </signal>
 <signal name="Y1">
@@
 <wire x1="32.623" y1="26.416" x2="32.623" y2="24.2824" width="0.3048" layer="1"/>
 <wire x1="32.623" y1="26.416" x2="28.94" y2="30.099" width="0.3048" layer="1"/>
-<wire x1="28.94" y1="30.099" x2="20.315" y2="30.099" width="0.3048" layer="1"/>
+<wire x1="28.94" y1="30.099" x2="20.265" y2="30.099" width="0.3048" layer="1"/>
 </signal>
 <signal name="G2">
@@
 <wire x1="28.559" y1="15.875" x2="22.59" y2="15.875" width="0.3048" layer="1"/>
 <wire x1="22.59" y1="15.875" x2="20.431" y2="18.034" width="0.3048" layer="1"/>
-<wire x1="20.431" y1="18.034" x2="20.315" y2="18.034" width="0.3048" layer="1"/>
+<wire x1="20.431" y1="18.034" x2="20.265" y2="18.034" width="0.3048" layer="1"/>
 </signal>
 <signal name="R2">
@@
 <wire x1="30.083" y1="14.986" x2="30.083" y2="18.1356" width="0.3048" layer="1"/>
 <wire x1="30.083" y1="14.986" x2="25.511" y2="10.414" width="0.3048" layer="1"/>
-<wire x1="25.511" y1="10.414" x2="20.315" y2="10.414" width="0.3048" layer="1"/>
+<wire x1="25.511" y1="10.414" x2="20.265" y2="10.414" width="0.3048" layer="1"/>
 </signal>
 <signal name="Y2">
@@
 <wire x1="29.448" y1="19.685" x2="29.448" y2="15.367" width="0.2032" layer="1"/>
 <wire x1="29.448" y1="15.367" x2="28.305" y2="14.224" width="0.3048" layer="1"/>
-<wire x1="28.305" y1="14.224" x2="20.315" y2="14.224" width="0.3048" layer="1"/>
+<wire x1="28.305" y1="14.224" x2="20.265" y2="14.224" width="0.3048" layer="1"/>
 </signal>
 </signals>
